Commit message: Enable full seven-joint VR control
Remove the temporary right-wrist restrictions so both arms use symmetric wrist travel and all seven body joints during full-pose IK.

Co-authored-by: Cursor <cursoragent@cursor.com>

File: telegrip_teleoperation/URDF/dual_scorpion/dual_scorpion_right.urdf (robot description, URDF)
Before this commit: robot dual_scorpion_right, 10 links, 9 joints
Joints:
- joint joint6: limit lower=-0.0523599 upper=2.96706 effort=1 velocity=1 -> lower=-2.96706 upper=2.96706 effort=1 velocity=1
